Commit message: feat: ros2_control 하드웨어 플러그인·주기를 xacro 인자로 뽑는다 [S2]
플러그인이 mock_components/GenericSystem 으로 박혀 있어 실기로 갈아끼울 수 없었다.
매크로에 plugin·rw_rate·is_async 를 내고 3단(demo.launch.py mappings →
hcr_robot.urdf.xacro → hcr_robot.xacro → 매크로)으로 관통시켰다. 셋 다 기본값이
종전 거동이라 인자 없이 띄우면 지금과 똑같이 뜬다. 실기 전환은 인자 하나다 —
hardware_plugin:=hcr_bridge/HcrSystemInterface rw_rate:=30 is_async:=true

인자 이름은 동료 ysh 의 hcr5_description 과 글자까지 맞췄다(매크로 param=plugin,
최상위 xacro:arg=hardware_plugin). 나중 이식이 한 줄이 되게 하기 위함이고,
중간결과물 §4 가 적어 둔 use_mock 불리언은 폐기한다 — 어떤 플러그인을 로드하는지가
불리언으로 표현되지 않는다.

xacro:arg 선언을 hcr_robot.xacro 안에 둔 이유
이 URDF 를 읽는 진입점이 둘이다. hcr_robot_description/launch/display.launch.py 는
hcr_robot.xacro 를 직접 읽고, hcr_moveit_config 는 그것을 include 한다. 선언과
기본값을 이 파일 한 곳에 두어야 두 경로가 다 살고 기본값이 갈리지 않는다.

initial_value 를 URDF 홈으로 교체
[0,0,1.5669,-1.59,-1.4695,0] 은 폐기된 SRDF 값이었다 — 실기 홈에서 715mm 떨어진
자세다(업무목록 T16 ③). [1.570796,0,1.570796,0,1.570796,0] 으로 바꿨고 SRDF
hcr_home 과 일치한다.

demo.launch.py — OpaqueFunction
MoveItConfigsBuilder 는 호출되는 그 자리에서 xacro 를 전개한다. LaunchConfiguration
객체를 mappings 에 그냥 넣으면 문자열로 안 풀려 조용히 깨진다. OpaqueFunction 안에서
perform(context) 로 해소한 뒤 넘긴다. launch 인자 기본값은 빈 문자열이고, 비면
mappings 에서 빠져 xacro 기본값이 산다 — 기본값 원본을 한 곳에 두기 위함이다.

mock 회귀 DoD 7/7 통과 (ROS_DOMAIN_ID=2, ros2_control 4.45.2)
xacro 전개 4조합 · 컴포넌트 1개 active · 인터페이스 cmd 6/state position 6/velocity 6 ·
컨트롤러 2개 active · /joint_states 99.87Hz · 초기자세 오차 0.000000rad ·
MoveIt2 Plan&Execute error_code=1, 도달오차 0.000889rad.
상세와 S1 병합용 §4 두 행은 briefs/drafts/중간결과물_S2.md (루트 디렉터리, git 밖)

File: hanwha_robot_arm/HCR_5/hcr_moveit_config/config/hcr_robot.urdf.xacro (robot description, xacro)
@@ -1,3 +1,9 @@
 <?xml version="1.0"?>
+<!--
+  MoveIt2 진입점. 인자 `hardware_plugin` · `rw_rate` · `is_async` 를 그대로 통과시킨다
+  (demo.launch.py 의 mappings → 여기 → hcr_robot.xacro → ros2_control 매크로).
+  선언과 기본값은 여기 두지 않는다 — 원본은 hcr_robot_description/urdf/hcr_robot.xacro
+  한 곳이고, display.launch.py 도 같은 선언을 쓴다. 두 곳에 두면 기본값이 갈린다.
+-->
 <robot xmlns:xacro="http://www.ros.org/wiki/xacro" name="hcr_robot">
   <xacro:include filename="$(find hcr_robot_description)/urdf/hcr_robot.xacro" />

File: hanwha_robot_arm/HCR_5/hcr_robot_description/urdf/hcr_robot.ros2_control.xacro (robot description, xacro)
@@ -1,13 +1,37 @@
 <?xml version="1.0"?>
 <robot xmlns:xacro="http://www.ros.org/wiki/xacro">
-  <xacro:macro name="hcr_robot_ros2_control" params="name:=hcr_robot_system">
-    <ros2_control name="${name}" type="system">
+  <!--
+    ══ 하드웨어 추상화 경계 ═══════════════════════════════════════════════════
+    sim 과 실기가 **같은 URDF 를 쓰고 플러그인만 갈아끼운다.** 셋 다 기본값이 있어
+    인자 없이 부르던 기존 사용처(display.launch.py · MoveIt2 demo)는 그대로 동작한다.
+      plugin    실기는 hcr_bridge/HcrSystemInterface.
+                인자명을 동료 ysh 의 hcr5_description 과 맞춰 이식을 한 줄로 뒀다
+      rw_rate   이 하드웨어 컴포넌트만의 read()/write() 주기(Hz).
+                controller_manager 의 update_rate 와 분리된다 (ros2_control 4.45.2).
+                기본 100 = update_rate 와 같은 값이라 mock 거동이 종전과 같다.
+                ⚠️ 파서가 양의 정수를 요구한다 — 0 을 기본값으로 두면 뜨지 않는다
+      is_async  실기 명령 RPC 왕복이 115~137ms 라 동기 발행은 100Hz 루프를 막는다.
+                워커 스레드로 분리할 때 true
+    실기 경로는 `rw_rate:=30 is_async:=true` 로 연다 — 상태 버스 실측이 29.1Hz 다.
+    근거: src/drivers/hcr_comm/ros2_control_hw_interface/중간결과물.md §2
+    ════════════════════════════════════════════════════════════════════════ -->
+  <xacro:macro name="hcr_robot_ros2_control"
+               params="name:=hcr_robot_system
+                       plugin:=mock_components/GenericSystem
+                       rw_rate:=100
+                       is_async:=false">
+    <ros2_control name="${name}" type="system" rw_rate="${rw_rate}" is_async="${is_async}">
       <hardware>
-        <plugin>mock_components/GenericSystem</plugin>
+        <plugin>${plugin}</plugin>
       </hardware>
+      <!-- initial_value = URDF 홈 [90, 0, 90, 0, 90, 0]°.
+           실기 홈 [0, −90, −90, −90, 90, 0]° 에 규약변환 q_URDF = s·q_실기 + δ 를
+           적용한 값이고 SRDF `hcr_home` 과 일치한다.
+           종전 값 [0, 0, 1.5669, −1.59, −1.4695, 0] 은 폐기된 SRDF 값이었다 —
+           실기 홈에서 715mm 떨어진 자세다. 근거: 업무목록 T16 ③ -->
       <joint name="joint_1">
         <command_interface name="position"/>
         <state_interface name="position">
-          <param name="initial_value">0</param>
+          <param name="initial_value">1.570796</param>
         </state_interface>
         <state_interface name="velocity"/>
@@ -23,5 +47,5 @@
         <command_interface name="position"/>
         <state_interface name="position">
-          <param name="initial_value">1.5669</param>
+          <param name="initial_value">1.570796</param>
         </state_interface>
         <state_interface name="velocity"/>
@@ -30,5 +54,5 @@
         <command_interface name="position"/>
         <state_interface name="position">
-          <param name="initial_value">-1.59</param>
+          <param name="initial_value">0</param>
         </state_interface>
         <state_interface name="velocity"/>
@@ -37,5 +61,5 @@
         <command_interface name="position"/>
         <state_interface name="position">
-          <param name="initial_value">-1.4695</param>
+          <param name="initial_value">1.570796</param>
         </state_interface>
         <state_interface name="velocity"/>

File: hanwha_robot_arm/HCR_5/hcr_robot_description/urdf/hcr_robot.xacro (robot description, xacro)
@@ -1,9 +1,23 @@
 <?xml version="1.0" ?>
 <robot name="hcr_robot" xmlns:xacro="http://www.ros.org/wiki/xacro">
+<!-- ── 인자 (하드웨어 추상화 경계) ────────────────────────────────────────────
+  선언을 **이 파일에** 두는 이유 — 이 URDF 를 읽는 진입점이 둘이다.
+    · hcr_robot_description/launch/display.launch.py  → 이 파일을 직접 읽는다
+    · hcr_moveit_config/config/hcr_robot.urdf.xacro   → 이 파일을 include 한다
+  기본값을 여기 두어야 두 경로가 다 산다. moveit 쪽에서 넘기는 mappings 가 이 기본값을 덮는다.
+    xacro hcr_robot.xacro                                          # mock (기본)
+    xacro hcr_robot.xacro hardware_plugin:=hcr_bridge/HcrSystemInterface \
+                          rw_rate:=30 is_async:=true               # 실기
+  값의 의미·근거는 hcr_robot.ros2_control.xacro 머리말 -->
+<xacro:arg name="hardware_plugin" default="mock_components/GenericSystem"/>
+<xacro:arg name="rw_rate"         default="100"/>
+<xacro:arg name="is_async"        default="false"/>
 <xacro:include filename="$(find hcr_robot_description)/urdf/materials.xacro" />
 <xacro:include filename="$(find hcr_robot_description)/urdf/hcr_robot.trans" />
 <xacro:include filename="$(find hcr_robot_description)/urdf/hcr_robot.gazebo" />
 <xacro:include filename="$(find hcr_robot_description)/urdf/hcr_robot.ros2_control.xacro" />
-<xacro:hcr_robot_ros2_control/>
+<xacro:hcr_robot_ros2_control plugin="$(arg hardware_plugin)"
+                              rw_rate="$(arg rw_rate)"
+                              is_async="$(arg is_async)"/>
 <link name="base_link">
   <inertial>
