Commit message: fix: URDF 를 실기 기구학에 맞춘다 — 정렬 안 돼 있었다 (RMS 43.4mm → 0.006mm)
실기 FK RPC(robot/convertPose)로 6축을 20°씩 전 회전 스윕(108샘플, 원적합 RMS
0.000mm)해 실기 기구학을 추출하고 이 URDF 와 대조한 결과다. 두 모델은 **영점 규약도
링크 치수도 달랐다**. 링크 치수가 틀리면 IK 가 그럴듯한 답을 내고 로봇이 조용히
4cm 엉뚱한 곳을 찍으므로, 관절한계(더미값)보다 위험한 결함이었다.

■ origin 교정 — joint_6.x 의 42.9mm 가 지배적
  joint_6.x  -0.089596 → -0.132498   (-42.90mm) ★ 이것만 고쳐도 43.4→1.6mm
  joint_3.z  +0.424    → +0.425001   (상완 +1mm)
  joint_3.y  +0.001    → 0
  joint_2.x  -0.0785   → -0.059138   ┐ 두 축이 평행해 합만 의미 있어 보이지만
  joint_3.x  +0.000652 → -0.019348   ┘ 사이에 J2 회전이 끼어 개별 식별된다
  joint_4.z  +0.338567 → +0.338499
  joint_5.z  +0.089596 → +0.089504
  → 109샘플 검증 RMS 0.0060mm, 최대 0.0130mm
  어깨 높이·전완·손목수직은 원래 0.1mm 이내로 맞았다. mesh 는 CAD 기준 그대로라
  시각화가 42.9mm 어긋난다 — 실기 제어에 기구학 일치가 우선이라 이쪽을 택했다.

■ 관절 규약 — 브릿지가 반드시 적용해야 한다
  q_URDF[i] = SIGN[i]*q_real[i] + DELTA[i]   (도)
  SIGN = (+1,+1,-1,+1,+1,+1)   DELTA = (90,90,0,90,0,0)
  실기 zero = 팔이 수평으로 뻗은 자세, URDF zero = 수직으로 선 자세.
  **변환을 빼먹으면 에러 없이 전혀 다른 자세로 간다.**

■ 관절한계 — CAD 더미값을 공식값으로 (실기_연결_현황.md §5)
  velocity 100 rad/s(=5729°/s, 공식의 32배) → 3.141593 (=180°/s, Appendix G)
  범위: ±360°, J3 만 ±165° (Appendix F). 종전 joint_1·6 은 0~360° 라 음수 방향이
  막혀 IK 해가 있어도 계획이 실패했고, joint_5 는 ±120° 라 **실기 현재 자세
  (wrist2 = -267°)조차 표현 못 했다**.
  joint_limits.yaml 의 max_acceleration 3.0 은 추정값이다 — 공식 매뉴얼에 항목이
  없어 Appendix G 정지거리에서 역산했다. 벤더 확인 대상.

■ SRDF hcr_home 교체
  종전 (0,0,1.5669,-1.59,-1.4695,0) 은 실기 홈에서 715mm 떨어진 자세로, 근거 없이
  들어간 값으로 보인다. 실기 홈 [0,-90,-90,-90,90,0](Mark 확인) = URDF
  [90,0,90,0,90,0]. 이 자세의 flange 는 (490.0,-170.5,441.5) rx=-180 으로 플랜지가
  정확히 아래를 향한다 — 소묘 기준자세로 그대로 쓸 수 있다.

근거·재현 절차: 업무목록 T16 · T1

File: hanwha_robot_arm/HCR_5/hcr_robot_description/urdf/hcr_robot.xacro (robot description, xacro)
@@ -146,4 +146,21 @@
   </collision>
 </link>
+<!-- ═══ 2026-08-05 실측 교정 ═══════════════════════════════════════════════════
+  실기(Rodi 1.003.005)의 FK RPC robot/convertPose 로 6축을 20°씩 전 회전 스윕(108샘플,
+  원적합 RMS 0.000mm)해 기구학을 추출하고 이 URDF 와 대조했다. 결과:
+  · origin 이 실기와 달랐다 (아래 ★ 표시 8곳). 특히 joint_6.x 의 42.9mm 오차가 지배적으로,
+    그것만 고쳐도 RMS 43.4mm → 1.6mm 로 떨어진다. 나머지는 1mm 이하의 미세 보정이다.
+    전부 적용 후 전 자세 위치오차 **RMS 43.4mm → 0.0060mm** (최대 0.0130mm, 109샘플 검증).
+  · limit 은 CAD 더미값(velocity=100 rad/s = 5729°/s)이었다. 매뉴얼 공식값으로 교체.
+  · 실기와 URDF 는 **영점 규약이 다르다**. 브릿지는 반드시 아래 변환을 적용할 것:
+        q_URDF[i] = s[i]*q_실기[i] + δ[i]      (도)
+        s = (+1, +1, −1, +1, +1, +1)          ← J3 만 부호 반전
+        δ = ( 90,  90,   0,  90,   0,   0)
+    실기 zero = 팔이 수평으로 뻗은 자세, URDF zero = 팔이 수직으로 선 자세.
+    실기 홈 [0,−90,−90,−90,90,0] = URDF [90,0,90,0,90,0] (SRDF hcr_home 과 일치시킴)
+  · mesh 는 CAD 기준 그대로다 — joint_6 을 42.9mm 옮겼으므로 시각화가 그만큼 어긋난다.
+    실기 제어에는 기구학 일치가 우선이라 이쪽을 택했다. mesh 교체는 별도 과제.
+  근거·재현: 업무목록 T16 · src/drivers/hcr_comm/README.md
+════════════════════════════════════════════════════════════════════════════ -->
 <joint name="joint_1" type="revolute">
   <origin xyz="0.0 0.0 0.03" rpy="0 0 0"/>
@@ -151,40 +168,52 @@
   <child link="link1_1"/>
   <axis xyz="0.0 -0.0 1.0"/>
-  <limit upper="6.283185" lower="0.0" effort="100" velocity="100"/>
+  <!-- 공식 ±360°, 180°/s (Appendix F·G). 종전 0~360°(음수 불가)는 IK 해가 있어도 계획 실패를 낳았다 -->
+  <limit upper="6.283185" lower="-6.283185" effort="100" velocity="3.141593"/>
 </joint>
 <joint name="joint_2" type="revolute">
-  <origin xyz="-0.0785 0.0 0.118778" rpy="0 0 0"/>
+  <!-- ★ 실측 교정: x −0.0785→−0.059138 (+19.36mm). joint_3.x 와 짝을 이룬다 (아래 참조) -->
+  <origin xyz="-0.059138 0.0 0.119001" rpy="0 0 0"/>
   <parent link="link1_1"/>
   <child link="link2_1"/>
   <axis xyz="-1.0 0.0 0.0"/>
-  <limit upper="1.570796" lower="-1.570796" effort="100" velocity="100"/>
+  <limit upper="6.283185" lower="-6.283185" effort="100" velocity="3.141593"/>
 </joint>
 <joint name="joint_3" type="revolute">
-  <origin xyz="0.000652 0.001 0.424" rpy="0 0 0"/>
+  <!-- ★ 실측 교정: z 0.424→0.425001 (상완 +1mm) · y 0.001→0 · x 0.000652→−0.019348
+       joint_2.x 와 joint_3.x 는 축이 평행해 겉보기엔 합만 의미 있을 것 같지만, 두 origin
+       사이에 J2 회전이 끼어 있어 실제로는 개별 식별된다. 합만 맞추면 RMS 가 0.28mm 로
+       남고, 최소제곱 해를 그대로 쓰면 0.0038mm 가 된다 -->
+  <origin xyz="-0.019348 0.0 0.425001" rpy="0 0 0"/>
   <parent link="link2_1"/>
   <child link="link3_1"/>
   <axis xyz="1.0 0.0 0.0"/>
-  <limit upper="2.268928" lower="-2.268928" effort="100" velocity="100"/>
+  <!-- J3 만 별도 제한 ±165° 가 실제로 존재한다 -->
+  <limit upper="2.879793" lower="-2.879793" effort="100" velocity="3.141593"/>
 </joint>
 <joint name="joint_4" type="revolute">
-  <origin xyz="-0.030016 -8e-06 0.338567" rpy="0 0 0"/>
+  <!-- ★ 실측 교정: z 0.338567→0.338499 (−0.07mm) -->
+  <origin xyz="-0.030016 -8e-06 0.338499" rpy="0 0 0"/>
   <parent link="link3_1"/>
   <child link="link4_1"/>
   <axis xyz="-1.0 0.0 -0.0"/>
-  <limit upper="2.96706" lower="-2.96706" effort="100" velocity="100"/>
+  <limit upper="6.283185" lower="-6.283185" effort="100" velocity="3.141593"/>
 </joint>
 <joint name="joint_5" type="revolute">
-  <origin xyz="-0.062 0.0 0.089596" rpy="0 0 0"/>
+  <!-- ★ 실측 교정: z 0.089596→0.089504 (−0.09mm) -->
+  <origin xyz="-0.062 0.0 0.089504" rpy="0 0 0"/>
   <parent link="link4_1"/>
   <child link="link5_1"/>
   <axis xyz="-0.0 -0.0 1.0"/>
-  <limit upper="2.094395" lower="-2.094395" effort="100" velocity="100"/>
+  <!-- 실기 wrist2 가 −267° 로 관측된다 — 종전 ±120° 로는 현재 자세조차 표현 못 했다 -->
+  <limit upper="6.283185" lower="-6.283185" effort="100" velocity="3.141593"/>
 </joint>
 <joint name="joint_6" type="revolute">
-  <origin xyz="-0.089596 0.0 0.062" rpy="0 0 0"/>
+  <!-- ★ 실측 교정: x −0.089596→−0.132498 (−42.90mm). J5 축에서 flange 까지 거리가
+       실기 132.5mm 인데 URDF 는 89.6mm 였다. 이 한 건이 전체 오차의 대부분이었다 -->
+  <origin xyz="-0.132498 0.0 0.062" rpy="0 0 0"/>
   <parent link="link5_1"/>
   <child link="link6_1"/>
   <axis xyz="-1.0 -0.0 0.0"/>
-  <limit upper="6.283185" lower="0.0" effort="100" velocity="100"/>
+  <limit upper="6.283185" lower="-6.283185" effort="100" velocity="3.141593"/>
 </joint>
 </robot>

Commit message: fix(urdf): joint_1·2·4 한계가 실기 가동범위와 90° 어긋나 있었다 — δ=90° 미반영 (T15·T16)
URDF 한계가 URDF 좌표에서 **대칭 ±360°** 로 박혀 있었는데, 규약 변환
q_URDF = s·q_실기 + δ 의 δ=90° 가 붙는 j1·j2·j4 는 그 대칭이 실기에서 깨진다:

  upper +360°(6.283185)  → 실기 **+270°**  ← 공식 +360° 보다 90° 좁다
  lower −360°(−6.283185) → 실기 **−450°**  ← 공식 −360° 보다 90° 넓다

양(+)방향으로 **한 바퀴를 못 돌았다.** 03pc 에서 액션 직송으로 발견했다 — joint_1
목표가 6.2832rad(= 실기 270°)에 닿자 하드웨어 게이트가 발행을 끊었고 로봇이 **실기
267.77°** 에 섰다. 음(−)방향 초과분은 `withinLimits()` 가 실기 ±360° 로 따로 막고
있었으므로 **안전에는 구멍이 없었다** — 못 가는 쪽만 문제였다.

→ j1·j2·j4 를 실기 ±360° 정합값으로 바꾼다. upper `7.853981` · lower `-4.712388`.
  j3(δ=0 · ±165°) · j5 · j6(δ=0 · ±360°) 는 δ=0 이라 어긋나지 않아 손대지 않았다.

⚠️ 끝자리를 **안쪽으로 내렸다.** 정확한 450° 는 7.853981633974483 이라, 반올림한
  `7.853982` 를 쓰면 실기 환산이 360.000021° 가 되어 `withinLimits()` 에 걸린다 —
  URDF 검사는 통과하는데 실기 검사가 막는 **게이트 충돌**이다. 첫 수정에서 실제로
  목표 360° 가 차단돼 359.98° 에 멈췄다. URDF 한계는 실기보다 항상 안쪽에 둔다.

실증 (03pc · 2°/s · 엔드이펙터 제거): 홈 0° → 280° → 360° → 0° 완주. 280° 로 종전
벽 270° 통과, 360° 지점 flange (489.941, −170.671, 441.500) 가 홈 (490.0, −170.5,
441.5) 과 일치 — 제자리 한 바퀴를 기하학적으로 확인했다. 축온 최고 55°C (임계 58
미도달). 종료 시 홈 `-0.0000°` · 서보 OFF.

함정 기재는 `hcr_bridge/운전절차.md` §5 ⑨⑩.

File: hanwha_robot_arm/HCR_5/hcr_robot_description/urdf/hcr_robot.xacro (robot description, xacro)
@@ -189,5 +189,16 @@
   <axis xyz="0.0 -0.0 1.0"/>
   <!-- 공식 ±360°, 180°/s (Appendix F·G). 종전 0~360°(음수 불가)는 IK 해가 있어도 계획 실패를 낳았다 -->
-  <limit upper="6.283185" lower="-6.283185" effort="100" velocity="3.141593"/>
+  <!-- ★ 2026-08-15 교정 — 한계를 **실기 ±360° 에 정합**시켰다. 종전 URDF 대칭 ±360° 는
+       δ=90° 탓에 실기로는 [+270°, −450°] 라, 양(+)방향으로 **한 바퀴를 못 돌았다.**
+       실측: 실기 267.77° 에서 발행이 끊겼다 (URDF 360° = 실기 270° 벽).
+         upper  7.853981 ≈ URDF +450° = 실기 +360°
+         lower −4.712388 ≈ URDF −270° = 실기 −360°
+       ⚠️ 끝자리를 **안쪽으로 내렸다.** 정확한 450° 는 7.853981633974483 인데, 반올림한
+          `7.853982` 를 쓰면 실기 환산이 **360.000021°** 라 `withinLimits()`(실기 ±360°)에 걸린다 —
+          URDF 한계는 통과하는데 실기 검사가 막는 **게이트 충돌**이다. `-4.712389` 도 같다(−360.0000011°).
+          실측 2026-08-15: 목표 360° 가 이 경계에서 차단돼 **359.98° 에 멈췄다.**
+          URDF 한계는 실기 한계보다 **항상 안쪽**이어야 두 검사가 싸우지 않는다.
+       δ=90° 인 j1·j2·j4 가 같은 결함이었다. 근거: hcr_bridge/운전절차.md §5 함정 ⑨ -->
+  <limit upper="7.853981" lower="-4.712388" effort="100" velocity="3.141593"/>
 </joint>
 <joint name="joint_2" type="revolute">
@@ -197,5 +208,6 @@
   <child link="link2_1"/>
   <axis xyz="-1.0 0.0 0.0"/>
-  <limit upper="6.283185" lower="-6.283185" effort="100" velocity="3.141593"/>
+  <!-- ★ 2026-08-15 교정 — δ=90° 정합. joint_1 주석 참조 -->
+  <limit upper="7.853981" lower="-4.712388" effort="100" velocity="3.141593"/>
 </joint>
 <joint name="joint_3" type="revolute">
@@ -217,5 +229,6 @@
   <child link="link4_1"/>
   <axis xyz="-1.0 0.0 -0.0"/>
-  <limit upper="6.283185" lower="-6.283185" effort="100" velocity="3.141593"/>
+  <!-- ★ 2026-08-15 교정 — δ=90° 정합. joint_1 주석 참조 -->
+  <limit upper="7.853981" lower="-4.712388" effort="100" velocity="3.141593"/>
 </joint>
 <joint name="joint_5" type="revolute">
