Commit message: chore: markch/hcr5_ros2 의 실측 자산을 로컬에 반입
우리가 만든 것이 아니라 **팀원 브랜치에서 그대로 가져온 것**이다. 로컬에서
돌려보려면 필요해서 반입했다. markch/hcr5_ros2 가 main 에 병합되면 이 커밋은
불필요해지므로, push 할 때 뺄 수 있도록 우리 작업과 분리해 둔다.

  hanwha_robot_arm/  URDF·SRDF·joint_limits·ros2_control (7 파일)
    · 관절 위치 한계를 실측/공식값으로 (관절 6 개 ±360°, joint_3 만 ±165°)
    · max_velocity 100 → 3.141593 rad/s (매뉴얼 Appendix G, 180°/s)
    · 실기 FK 108 샘플 스윕으로 링크 원점 교정 (위치오차 RMS 43.4mm → 0.006mm)
    · hcr_home 재정의 (joint_1 0° → +90°)

  src/drivers/nyang_pen/  펜홀더 + pen_tip TCP 프레임 패키지
    · tool0 → holder → body → pen_tip 체인
    · 치수는 명목값. 실측하면 macro params 기본값만 갈아끼운다

⚠️ URDF 숫자를 그대로 각도로 읽으면 오해한다. joint_1 의 [-4.712388, 7.853981]
   은 [-270°, +450°] 로 읽히지만 ±360° 를 90° 민 표기다 (폭 720° 로 동일).
   실기 각도와 URDF 기준점이 90° 어긋나 있다.

⚠️ 컨테이너가 nyang_pen 을 찾으려면 워크스페이스 안에 있어야 해서
   ws_moveit2/src/ 와 ws_simulation/src/ 에 사본을 뒀다. 그 둘은 .gitignore
   대상이다 — 정식 해법은 compose 에 바인드 마운트를 추가하는 것이다.

Co-Authored-By: Claude Opus 5 <noreply@anthropic.com>

File: hanwha_robot_arm/HCR_5/hcr_robot_description/urdf/hcr_robot.ros2_control.xacro (robot description, xacro)
@@ -2,20 +2,55 @@
 <robot xmlns:xacro="http://www.ros.org/wiki/xacro">
   <!--
-    하드웨어 플러그인을 인자로 받는다 (기본값은 종전과 같은 mock).
-    이것이 SA 가 말하는 하드웨어 추상화 경계(N6·F7.3)의 실제 구현 지점이다 —
-    시뮬레이션·실물이 **같은 URDF 로 플러그인만 갈아끼운다.** 기본값을 두었으므로
-    이 매크로를 그냥 호출하던 기존 사용처(MoveIt2 demo 등)는 달라지지 않는다.
-    예: <xacro:hcr_robot_ros2_control plugin="mujoco_ros2_control/MujocoSystemInterface"/>
-  -->
+    ══ 하드웨어 추상화 경계 ═══════════════════════════════════════════════════
+    sim 과 실기가 **같은 URDF 를 쓰고 플러그인만 갈아끼운다.** 셋 다 기본값이 있어
+    인자 없이 부르던 기존 사용처(display.launch.py · MoveIt2 demo)는 그대로 동작한다.
+      plugin    실기는 hcr5_bridge/HcrSystemInterface.
+                인자명을 동료 ysh 의 hcr5_description 과 맞춰 이식을 한 줄로 뒀다
+      rw_rate   이 하드웨어 컴포넌트만의 read()/write() 주기(Hz).
+                controller_manager 의 update_rate 와 분리된다 (ros2_control 4.45.2).
+                기본 100 = update_rate 와 같은 값이라 mock 거동이 종전과 같다.
+                ⚠️ 파서가 양의 정수를 요구한다 — 0 을 기본값으로 두면 뜨지 않는다
+      is_async  실기 명령 RPC 왕복이 115~137ms 라 동기 발행은 100Hz 루프를 막는다.
+                워커 스레드로 분리할 때 true
+    앞의 셋은 `<ros2_control>` **속성**이고, 아래 둘은 `<hardware>` 안의 **`<param>`** 이다.
+    ros2_control 이 둘을 다른 자리에서 읽으므로 실리는 곳이 다르다.
+      allow_motion  실기를 **실제로 움직일지**의 안전 잠금. 플러그인 기본값이 false 이고
+                    이 param 만이 켜는 유일한 통로다 (hcr_system_interface.cpp:108-118).
+                    false 면 write() 가 무동작 — 실기 '읽기 전용' 모드가 이 상태다.
+                    ⚠️ true 는 로봇이 움직인다. 서보 ON·e-stop 대기·입회를 갖추고서만 쓴다
+      servo_off_on_deactivate
+                    비활성화(= 종료)될 때 서보를 끌지. **기본 true.**
+                    allow_motion 과 무관하게 적용된다 — 읽기 전용으로 띄웠어도 서보는
+                    launch 나 사람이 켜 뒀을 수 있기 때문이다. mock 플러그인은 이 param 을
+                    안 읽으므로 mock 거동은 종전과 같다.
+                    ⚠️ false 로 두면 종료 후 서보가 켜진 채 남는다 — 축온이 올라
+                    58~61°C 에서 6축이 트립한다(2026-08-05, 컨트롤러 재부팅으로만 복구).
+                    자세가 위험해 브레이크를 걸고 싶지 않을 때만 false
+    실기 읽기는 `rw_rate:=30 is_async:=true` 로 연다 — 상태 버스 실측이 29.1Hz 다.
+    실기 쓰기는 거기에 `allow_motion:=true` 를 더한다.
+    근거: src/drivers/hcr5_comm/guideline/중간결과물.md §2·§5
+    ════════════════════════════════════════════════════════════════════════ -->
   <xacro:macro name="hcr_robot_ros2_control"
-               params="name:=hcr_robot_system plugin:=mock_components/GenericSystem">
-    <ros2_control name="${name}" type="system">
+               params="name:=hcr_robot_system
+                       plugin:=mock_components/GenericSystem
+                       rw_rate:=100
+                       is_async:=false
+                       allow_motion:=false
+                       servo_off_on_deactivate:=true">
+    <ros2_control name="${name}" type="system" rw_rate="${rw_rate}" is_async="${is_async}">
       <hardware>
         <plugin>${plugin}</plugin>
+        <param name="allow_motion">${allow_motion}</param>
+        <param name="servo_off_on_deactivate">${servo_off_on_deactivate}</param>
       </hardware>
+      <!-- initial_value = URDF 홈 [90, 0, 90, 0, 90, 0]°.
+           실기 홈 [0, −90, −90, −90, 90, 0]° 에 규약변환 q_URDF = s·q_실기 + δ 를
+           적용한 값이고 SRDF `hcr_home` 과 일치한다.
+           종전 값 [0, 0, 1.5669, −1.59, −1.4695, 0] 은 폐기된 SRDF 값이었다 —
+           실기 홈에서 715mm 떨어진 자세다. 근거: 업무목록 T16 ③ -->
       <joint name="joint_1">
         <command_interface name="position"/>
         <state_interface name="position">
-          <param name="initial_value">0</param>
+          <param name="initial_value">1.570796</param>
         </state_interface>
         <state_interface name="velocity"/>
@@ -31,5 +66,5 @@
         <command_interface name="position"/>
         <state_interface name="position">
-          <param name="initial_value">1.5669</param>
+          <param name="initial_value">1.570796</param>
         </state_interface>
         <state_interface name="velocity"/>
@@ -38,5 +73,5 @@
         <command_interface name="position"/>
         <state_interface name="position">
-          <param name="initial_value">-1.59</param>
+          <param name="initial_value">0</param>
         </state_interface>
         <state_interface name="velocity"/>
@@ -45,5 +80,5 @@
         <command_interface name="position"/>
         <state_interface name="position">
-          <param name="initial_value">-1.4695</param>
+          <param name="initial_value">1.570796</param>
         </state_interface>
         <state_interface name="velocity"/>

File: hanwha_robot_arm/HCR_5/hcr_robot_description/urdf/hcr_robot.xacro (robot description, xacro)
@@ -1,21 +1,31 @@
 <?xml version="1.0" ?>
 <robot name="hcr_robot" xmlns:xacro="http://www.ros.org/wiki/xacro">
+<!-- ── 인자 (하드웨어 추상화 경계) ────────────────────────────────────────────
+  선언을 **이 파일에** 두는 이유 — 이 URDF 를 읽는 진입점이 둘이다.
+    · hcr_robot_description/launch/display.launch.py  → 이 파일을 직접 읽는다
+    · hcr_moveit_config/config/hcr_robot.urdf.xacro   → 이 파일을 include 한다
+  기본값을 여기 두어야 두 경로가 다 산다. moveit 쪽에서 넘기는 mappings 가 이 기본값을 덮는다.
+    xacro hcr_robot.xacro                                          # mock (기본)
+    xacro hcr_robot.xacro hardware_plugin:=hcr5_bridge/HcrSystemInterface \
+                          rw_rate:=30 is_async:=true               # 실기 읽기
+    xacro hcr_robot.xacro hardware_plugin:=hcr5_bridge/HcrSystemInterface \
+                          rw_rate:=30 is_async:=true \
+                          allow_motion:=true                       # 실기 쓰기 ⚠️ 움직인다
+  값의 의미·근거는 hcr_robot.ros2_control.xacro 머리말 -->
+<xacro:arg name="hardware_plugin" default="mock_components/GenericSystem"/>
+<xacro:arg name="rw_rate"         default="100"/>
+<xacro:arg name="is_async"        default="false"/>
+<!-- 기본값 false 는 플러그인 기본값과 같다 — 인자를 잊어도 로봇은 안 움직인다 -->
+<xacro:arg name="allow_motion"    default="false"/>
+<xacro:arg name="servo_off_on_deactivate" default="true"/>
 <xacro:include filename="$(find hcr_robot_description)/urdf/materials.xacro" />
 <xacro:include filename="$(find hcr_robot_description)/urdf/hcr_robot.trans" />
 <xacro:include filename="$(find hcr_robot_description)/urdf/hcr_robot.gazebo" />
-<!--
-  ros2_control 블록 생성 여부와 하드웨어 플러그인을 인자로 받는다.
-  **기본값은 종전과 같다** — 인자 없이 include 하던 곳(MoveIt2 config 등)은 그대로 동작한다.
-    ros2_control:=false      블록을 만들지 않는다. 감싸는 쪽이 자체 블록을 정의할 때
-                             (시뮬레이션은 hardware 에 <param> 을 넣어야 해서 이 경로를 쓴다)
-    hardware_plugin:=<이름>  플러그인 교체 (실물 드라이버·MuJoCo 등)
-  이 갈래가 없으면 mock 블록이 **항상** 들어가 다른 하드웨어와 같은 조인트를 두고 충돌한다.
--->
-<xacro:arg name="ros2_control" default="true"/>
-<xacro:arg name="hardware_plugin" default="mock_components/GenericSystem"/>
 <xacro:include filename="$(find hcr_robot_description)/urdf/hcr_robot.ros2_control.xacro" />
-<xacro:if value="$(arg ros2_control)">
-  <xacro:hcr_robot_ros2_control plugin="$(arg hardware_plugin)"/>
-</xacro:if>
+<xacro:hcr_robot_ros2_control plugin="$(arg hardware_plugin)"
+                              rw_rate="$(arg rw_rate)"
+                              is_async="$(arg is_async)"
+                              allow_motion="$(arg allow_motion)"
+                              servo_off_on_deactivate="$(arg servo_off_on_deactivate)"/>
 <link name="base_link">
   <inertial>
@@ -158,4 +168,21 @@
   </collision>
 </link>
+<!-- ═══ 2026-08-05 실측 교정 ═══════════════════════════════════════════════════
+  실기(Rodi 1.003.005)의 FK RPC robot/convertPose 로 6축을 20°씩 전 회전 스윕(108샘플,
+  원적합 RMS 0.000mm)해 기구학을 추출하고 이 URDF 와 대조했다. 결과:
+  · origin 이 실기와 달랐다 (아래 ★ 표시 8곳). 특히 joint_6.x 의 42.9mm 오차가 지배적으로,
+    그것만 고쳐도 RMS 43.4mm → 1.6mm 로 떨어진다. 나머지는 1mm 이하의 미세 보정이다.
+    전부 적용 후 전 자세 위치오차 **RMS 43.4mm → 0.0060mm** (최대 0.0130mm, 109샘플 검증).
+  · limit 은 CAD 더미값(velocity=100 rad/s = 5729°/s)이었다. 매뉴얼 공식값으로 교체.
+  · 실기와 URDF 는 **영점 규약이 다르다**. 브릿지는 반드시 아래 변환을 적용할 것:
+        q_URDF[i] = s[i]*q_실기[i] + δ[i]      (도)
+        s = (+1, +1, −1, +1, +1, +1)          ← J3 만 부호 반전
+        δ = ( 90,  90,   0,  90,   0,   0)
+    실기 zero = 팔이 수평으로 뻗은 자세, URDF zero = 팔이 수직으로 선 자세.
+    실기 홈 [0,−90,−90,−90,90,0] = URDF [90,0,90,0,90,0] (SRDF hcr_home 과 일치시킴)
+  · mesh 는 CAD 기준 그대로다 — joint_6 을 42.9mm 옮겼으므로 시각화가 그만큼 어긋난다.
+    실기 제어에는 기구학 일치가 우선이라 이쪽을 택했다. mesh 교체는 별도 과제.
+  근거·재현: 업무목록 T16 · src/drivers/hcr5_mqtt/README.md
+════════════════════════════════════════════════════════════════════════════ -->
 <joint name="joint_1" type="revolute">
   <origin xyz="0.0 0.0 0.03" rpy="0 0 0"/>
@@ -163,40 +190,74 @@
   <child link="link1_1"/>
   <axis xyz="0.0 -0.0 1.0"/>
-  <limit upper="6.283185" lower="0.0" effort="100" velocity="100"/>
+  <!-- 공식 ±360°, 180°/s (Appendix F·G). 종전 0~360°(음수 불가)는 IK 해가 있어도 계획 실패를 낳았다 -->
+  <!-- ★ 2026-08-15 교정 — 한계를 **실기 ±360° 에 정합**시켰다. 종전 URDF 대칭 ±360° 는
+       δ=90° 탓에 실기로는 [+270°, −450°] 라, 양(+)방향으로 **한 바퀴를 못 돌았다.**
+       실측: 실기 267.77° 에서 발행이 끊겼다 (URDF 360° = 실기 270° 벽).
+         upper  7.853981 ≈ URDF +450° = 실기 +360°
+         lower −4.712388 ≈ URDF −270° = 실기 −360°
+       ⚠️ 끝자리를 **안쪽으로 내렸다.** 정확한 450° 는 7.853981633974483 인데, 반올림한
+          `7.853982` 를 쓰면 실기 환산이 **360.000021°** 라 `withinLimits()`(실기 ±360°)에 걸린다 —
+          URDF 한계는 통과하는데 실기 검사가 막는 **게이트 충돌**이다. `-4.712389` 도 같다(−360.0000011°).
+          실측 2026-08-15: 목표 360° 가 이 경계에서 차단돼 **359.98° 에 멈췄다.**
+          URDF 한계는 실기 한계보다 **항상 안쪽**이어야 두 검사가 싸우지 않는다.
+       δ=90° 인 j1·j2·j4 가 같은 결함이었다. 근거: hcr5_bridge/운전절차.md §5 함정 ⑨ -->
+  <limit upper="7.853981" lower="-4.712388" effort="100" velocity="3.141593"/>
 </joint>
 <joint name="joint_2" type="revolute">
-  <origin xyz="-0.0785 0.0 0.118778" rpy="0 0 0"/>
+  <!-- ★ 실측 교정: x −0.0785→−0.059138 (+19.36mm). joint_3.x 와 짝을 이룬다 (아래 참조) -->
+  <origin xyz="-0.059138 0.0 0.119001" rpy="0 0 0"/>
   <parent link="link1_1"/>
   <child link="link2_1"/>
   <axis xyz="-1.0 0.0 0.0"/>
-  <limit upper="1.570796" lower="-1.570796" effort="100" velocity="100"/>
+  <!-- ★ 2026-08-15 교정 — δ=90° 정합. joint_1 주석 참조 -->
+  <limit upper="7.853981" lower="-4.712388" effort="100" velocity="3.141593"/>
 </joint>
 <joint name="joint_3" type="revolute">
-  <origin xyz="0.000652 0.001 0.424" rpy="0 0 0"/>
+  <!-- ★ 실측 교정: z 0.424→0.425001 (상완 +1mm) · y 0.001→0 · x 0.000652→−0.019348
+       joint_2.x 와 joint_3.x 는 축이 평행해 겉보기엔 합만 의미 있을 것 같지만, 두 origin
+       사이에 J2 회전이 끼어 있어 실제로는 개별 식별된다. 합만 맞추면 RMS 가 0.28mm 로
+       남고, 최소제곱 해를 그대로 쓰면 0.0038mm 가 된다 -->
+  <origin xyz="-0.019348 0.0 0.425001" rpy="0 0 0"/>
   <parent link="link2_1"/>
   <child link="link3_1"/>
   <axis xyz="1.0 0.0 0.0"/>
-  <limit upper="2.268928" lower="-2.268928" effort="100" velocity="100"/>
+  <!-- J3 만 별도 제한 ±165° 가 실제로 존재한다 -->
+  <limit upper="2.879793" lower="-2.879793" effort="100" velocity="3.141593"/>
 </joint>
 <joint name="joint_4" type="revolute">
-  <origin xyz="-0.030016 -8e-06 0.338567" rpy="0 0 0"/>
+  <!-- ★ 실측 교정: z 0.338567→0.338499 (−0.07mm) -->
+  <origin xyz="-0.030016 -8e-06 0.338499" rpy="0 0 0"/>
   <parent link="link3_1"/>
   <child link="link4_1"/>
   <axis xyz="-1.0 0.0 -0.0"/>
-  <limit upper="2.96706" lower="-2.96706" effort="100" velocity="100"/>
+  <!-- ★ 2026-08-15 교정 — δ=90° 정합. joint_1 주석 참조 -->
+  <limit upper="7.853981" lower="-4.712388" effort="100" velocity="3.141593"/>
 </joint>
 <joint name="joint_5" type="revolute">
-  <origin xyz="-0.062 0.0 0.089596" rpy="0 0 0"/>
+  <!-- ★ 실측 교정: z 0.089596→0.089504 (−0.09mm) -->
+  <origin xyz="-0.062 0.0 0.089504" rpy="0 0 0"/>
   <parent link="link4_1"/>
   <child link="link5_1"/>
   <axis xyz="-0.0 -0.0 1.0"/>
-  <limit upper="2.094395" lower="-2.094395" effort="100" velocity="100"/>
+  <!-- 실기 wrist2 가 −267° 로 관측된다 — 종전 ±120° 로는 현재 자세조차 표현 못 했다 -->
+  <limit upper="6.283185" lower="-6.283185" effort="100" velocity="3.141593"/>
 </joint>
 <joint name="joint_6" type="revolute">
-  <origin xyz="-0.089596 0.0 0.062" rpy="0 0 0"/>
+  <!-- ★ 실측 교정: x −0.089596→−0.132498 (−42.90mm). J5 축에서 flange 까지 거리가
+       실기 132.5mm 인데 URDF 는 89.6mm 였다. 이 한 건이 전체 오차의 대부분이었다 -->
+  <origin xyz="-0.132498 0.0 0.062" rpy="0 0 0"/>
   <parent link="link5_1"/>
   <child link="link6_1"/>
   <axis xyz="-1.0 -0.0 0.0"/>
-  <limit upper="6.283185" lower="0.0" effort="100" velocity="100"/>
-</joint>
+  <limit upper="6.283185" lower="-6.283185" effort="100" velocity="3.141593"/>
+</joint>
+<!-- ── 공구: 펜홀더 nyang_pen ─────────────────────────────────────────────────
+  플랜지(link6_1) 아래로 tool0 → 홀더 → 펜 → pen_tip 을 잇는다. pose goal 은
+  pen_tip 을 겨눈다 — 이 include 가 없으면 IK 가 **플랜지 기준**으로 풀린다.
+  본체와 분리된 패키지인 이유 · 명목 치수 · 강성 가정 · 축 방향 근거는 전부
+  src/drivers/nyang_pen/urdf/nyang_pen.xacro 머리말에 있다. 여기 옮겨 적지 않는다.
+  치수를 바꿀 때도 그 파일의 매크로 기본값만 고친다 (P1 판정 — 인자 관통 안 함).
+  ⚠️ 이 패키지는 compose.yml 이 src/drivers/ 를 마운트해야 컨테이너에서 보인다 -->
+<xacro:include filename="$(find nyang_pen)/urdf/nyang_pen.xacro"/>
+<xacro:nyang_pen parent="link6_1"/>
 </robot>
