Commit message: fix: MuJoCo 변환 함정 3건 해소 — 원본 인자화 · --no-fuse · actuator 정의
공식 mujoco_ros2_control_demos 예제에서 규약을 확인해 세 가지를 모두 풀었다.
씬이 로드되고 물리가 돌며 필압 센서가 접촉을 잡는 것까지 확인.

① 원본 hcr_robot.xacro 인자화 (hanwha 자산)
   - ros2_control:=false 로 블록 생성을 끄고 hardware_plugin:=<이름> 으로 교체
   - **기본값이 종전과 같아 MoveIt2 경로는 달라지지 않는다** (인자 없이 파싱하면
     여전히 mock_components/GenericSystem — 실측 확인)
   - SA 가 말한 하드웨어 추상화 경계(N6·F7.3)의 실제 구현 지점이며 moveit2 도
     결국 필요로 하는 개선이라 원본에 넣었다

② --no-fuse — 펜이 link6_1 에 병합되던 것 해소. pen_link·pen_tip body 가 살아남음

③ mjcf/mujoco_inputs.xml 신설, 변환기 -m 으로 전달
   - actuator 6 개 생성 (없으면 nu=0 이라 아무것도 제어되지 않는다)
   - 같은 파일의 default class="visual"/"collision" 이 직전 세션의
     "unknown default class 'visual'" 로드 실패 원인이었다
   - modify_element 로 관절 damping·frictionloss 부여

필압 측정 경로
   - 펜이 아니라 **종이에 site + touch 센서**를 두었다. 변환된 로봇 MJCF 를
     후처리할 필요가 없어 재현이 쉽다

씬 경로는 launch 파라미터가 아니라 URDF hardware <param name="mujoco_model"> 로
넘기는 규약이라 launch 를 그에 맞게 고쳤다.

검증: 씬 로드 body 12 · joint 6 · geom 22 · actuator 6 · sensor 1 /
물리 2초 안정(관절 오차 0.003 rad) / 접촉·필압 감지 확인

⚠️ 시뮬이 R2 를 정량적으로 드러냈다 — 4 mm 침투에 408 N (실제 연필은 1~5 N 대).
위치 제어 + 테이프 고정(z 완충 없음)이라는 설계 그대로의 결과이며,
접촉·강성 파라미터 튜닝이 다음 우선순위다.

File: hanwha_robot_arm/HCR_5/hcr_robot_description/urdf/hcr_robot.ros2_control.xacro (robot description, xacro)
@@ -1,8 +1,16 @@
 <?xml version="1.0"?>
 <robot xmlns:xacro="http://www.ros.org/wiki/xacro">
-  <xacro:macro name="hcr_robot_ros2_control" params="name:=hcr_robot_system">
+  <!--
+    하드웨어 플러그인을 인자로 받는다 (기본값은 종전과 같은 mock).
+    이것이 SA 가 말하는 하드웨어 추상화 경계(N6·F7.3)의 실제 구현 지점이다 —
+    시뮬레이션·실물이 **같은 URDF 로 플러그인만 갈아끼운다.** 기본값을 두었으므로
+    이 매크로를 그냥 호출하던 기존 사용처(MoveIt2 demo 등)는 달라지지 않는다.
+    예: <xacro:hcr_robot_ros2_control plugin="mujoco_ros2_control/MujocoSystemInterface"/>
+  -->
+  <xacro:macro name="hcr_robot_ros2_control"
+               params="name:=hcr_robot_system plugin:=mock_components/GenericSystem">
     <ros2_control name="${name}" type="system">
       <hardware>
-        <plugin>mock_components/GenericSystem</plugin>
+        <plugin>${plugin}</plugin>
       </hardware>
       <joint name="joint_1">

File: hanwha_robot_arm/HCR_5/hcr_robot_description/urdf/hcr_robot.xacro (robot description, xacro)
@@ -4,6 +4,18 @@
 <xacro:include filename="$(find hcr_robot_description)/urdf/hcr_robot.trans" />
 <xacro:include filename="$(find hcr_robot_description)/urdf/hcr_robot.gazebo" />
+<!--
+  ros2_control 블록 생성 여부와 하드웨어 플러그인을 인자로 받는다.
+  **기본값은 종전과 같다** — 인자 없이 include 하던 곳(MoveIt2 config 등)은 그대로 동작한다.
+    ros2_control:=false      블록을 만들지 않는다. 감싸는 쪽이 자체 블록을 정의할 때
+                             (시뮬레이션은 hardware 에 <param> 을 넣어야 해서 이 경로를 쓴다)
+    hardware_plugin:=<이름>  플러그인 교체 (실물 드라이버·MuJoCo 등)
+  이 갈래가 없으면 mock 블록이 **항상** 들어가 다른 하드웨어와 같은 조인트를 두고 충돌한다.
+-->
+<xacro:arg name="ros2_control" default="true"/>
+<xacro:arg name="hardware_plugin" default="mock_components/GenericSystem"/>
 <xacro:include filename="$(find hcr_robot_description)/urdf/hcr_robot.ros2_control.xacro" />
-<xacro:hcr_robot_ros2_control/>
+<xacro:if value="$(arg ros2_control)">
+  <xacro:hcr_robot_ros2_control plugin="$(arg hardware_plugin)"/>
+</xacro:if>
 <link name="base_link">
   <inertial>

File: src/simulation/ws_simulation/src/sim_bringup/urdf/hcr_robot_pen.xacro (robot description, xacro)
@@ -11,19 +11,27 @@
 <robot name="hcr_robot_pen" xmlns:xacro="http://www.ros.org/wiki/xacro">
   <!--
-    원본 로봇 — **`hcr_robot.xacro` 가 아니라 플랫 URDF 를 가져온다.**
-    이유: `hcr_robot.xacro` 는 8행에서 `<xacro:hcr_robot_ros2_control/>` 를
-    **무조건** 호출해 `mock_components/GenericSystem` 블록을 만든다. 그것을
-    include 하면 mock 과 MuJoCo 하드웨어가 한 URDF 에 둘 다 들어가 같은 조인트를
-    두 시스템이 요구하게 된다. 플랫 URDF 에는 ros2_control 블록이 없어 이 충돌이 없다.
-    덤으로 플랫 쪽에는 `world` 링크와 base_link 를 고정하는 조인트가 있어
-    시뮬에서 로봇이 바닥에 붙는다 (xacro 쪽에는 없다).
-    ⚠️ ROS1 잔재인 `<transmission>`·`<gazebo>` 태그가 14 개 딸려온다. ROS 2 와
-    MuJoCo 변환기는 무시하지만, 원본을 정리할 때 함께 걷어낼 대상이다.
-    ⚠️ **근본 해결은 원본이 하드웨어 플러그인을 인자로 받게 하는 것**이다
-    (`use_mock_hardware` 같은 인자). moveit2 도 결국 sim/real 스위칭이 필요하므로
-    프로젝트 전체가 필요로 하는 개선이며, hanwha 자산 수정이라 별도 과제로 둔다 —
-    업무목록 참조.
+    ⚠️ **`ros2_control:=false` 를 이 줄들보다 먼저 선언해야 한다.**
+    xacro 의 `<xacro:arg>` 는 "아직 정의되지 않았으면 기본값을 넣는다"이므로,
+    여기서 먼저 false 를 박아 두면 include 되는 원본의 기본값(true)이 무시된다.
+    원본이 mock 블록을 만들지 않게 해서, 아래에서 MuJoCo 블록을 직접 정의한다.
   -->
-  <xacro:include filename="$(find hcr_robot_description)/urdf/hcr_robot_urdf.urdf"/>
+  <xacro:arg name="ros2_control" default="false"/>
+  <!-- MuJoCo 가 로드할 씬. **변환 산출물이라 git 제외 영역에 생긴다** —
+       robot_description_to_mjcf.sh 의 -o 로 지정한 곳과 맞춰야 한다. -->
+  <xacro:arg name="mujoco_scene" default="/home/rosuser/data/mjcf/scene.xml"/>
+  <xacro:arg name="headless" default="false"/>
+  <!-- 원본 로봇 (링크 7 · 조인트 6, inertial 전부 있음 — MuJoCo 변환 가능) -->
+  <xacro:include filename="$(find hcr_robot_description)/urdf/hcr_robot.xacro"/>
+  <!--
+    로봇을 월드에 고정한다. 원본 xacro 에는 world 링크가 없고 플랫 URDF 에만 있다 —
+    시뮬에서는 베이스가 떠 있으면 안 되므로 여기서 붙인다.
+    BRD §2.3: 철제 책상 상판에 수평 고정.
+  -->
+  <link name="world"/>
+  <joint name="world_to_base" type="fixed">
+    <parent link="world"/>
+    <child link="base_link"/>
+    <origin xyz="0 0 0" rpy="0 0 0"/>
+  </joint>
   <!-- ── 펜 ────────────────────────────────────────────────────────────────
        Phase 1 은 펜을 **테이프로 플랜지에 고정**한다 (BRD §2.3). 즉 z 방향
@@ -76,4 +84,10 @@
     <hardware>
       <plugin>mujoco_ros2_control/MujocoSystemInterface</plugin>
+      <!-- 씬은 launch 파라미터가 아니라 **여기 hardware param 으로** 넘긴다
+           (mujoco_ros2_control 규약 — demos 의 test_robot.urdf 와 같은 방식) -->
+      <param name="mujoco_model">$(arg mujoco_scene)</param>
+      <!-- true 면 Simulate 창을 띄우지 않는다. 확인 경로가 SVG 라 headless 로도 결과가 나온다 -->
+      <param name="headless">$(arg headless)</param>
+      <param name="sim_speed_factor">1.0</param>
     </hardware>
     <xacro:macro name="mujoco_joint" params="name initial">

Commit message: fix: 머지 b8ac9b9 에서 소실된 xacro 2개·.gitignore 를 복구한다
b8ac9b9 ("Merge branch 'main' into markch/hcr5_ros2") 가 충돌 파일 3개를
**양쪽 부모 어느 쪽도 아닌 상태**로 해소해 내용이 사라졌다. PR #6 이 그대로
main 에 실려 현재 origin/main 은 URDF 가 깨져 있다.

  파일                          베이스  hcr5_ros2   main  머지결과
  hcr_robot.xacro                 7422    14296     8299      1  ← 개행만 남음
  hcr_robot.ros2_control.xacro    1847     5609     2399   2077
  .gitignore                       808     1872     1514    614

■ 무엇이 깨졌나
  · hcr_robot.xacro 가 1 바이트라 이를 읽는 3곳이 전부 죽는다
      hcr_moveit_config/config/hcr_robot.urdf.xacro:9   (MoveIt2 진입점)
      hcr_robot_description/launch/display.launch.py:9
      src/drivers/hcr5_bridge/launch/bringup.launch.py:70
  · .gitignore 에서 **/compose.override.yml 이 사라져 PC 로컬 GPU 설정이
    `git add -A` 한 번에 팀 리포로 넘어갈 수 있었다.
    4c16830 이 막아 둔 구멍이 다시 열린 것 — 유출 여부는 확인했고, 없다.

■ 되살린 것 (커밋 7개 분량)
  6846588  URDF 실기 기구학 정렬 (RMS 43.4mm → 0.006mm)
  fcab110  하드웨어 플러그인·rw_rate·is_async 인자화 [S2]
  cc5a319  allow_motion 안전 잠금 관통 [S5]
  453b6c7  펜홀더 nyang_pen TCP 좌표계 [P1]
  a9d5f3e  joint_1·2·4 한계 δ=90° 교정 (T15·T16)
  f3fd572·6cef08a  서보 OFF 를 on_deactivate 로

■ 합친 방식 — 한쪽을 고르지 않고 양쪽 부모의 합집합을 만들었다
  · ros2_control.xacro : hcr5_ros2 쪽 그대로. main 이 04b83c9 에서 넣은
    plugin 인자는 이쪽 6-인자 매크로에 이미 들어 있다
  · hcr_robot.xacro    : hcr5_ros2 쪽 + main 의 ros2_control:=true/false 스위치.
    시뮬이 이 인자를 쓴다 (sim_bringup/urdf/hcr_robot_pen.xacro:21)
  · .gitignore         : hcr5_ros2 쪽 + main 의 data/ 3줄.
    main 의 개별 compose.override.yml 2줄은 **/compose.override.yml 글롭에 흡수된다

■ 검증
  xacro 파싱 5 갈래 (jazzy 컨테이너)
    ① 기본(mock)           OK  링크11·조인트22·블록1·mock·rw100·async False
    ② ros2_control:=false  OK  ros2_control 블록 0 (시뮬 경로)
    ③ 실기 읽기            OK  HcrSystemInterface·rw30·async True·allow_motion False
    ④ 실기 쓰기            OK  allow_motion True
    ⑤ MoveIt2 진입점       OK  링크11·블록1
  git check-ignore 13/13 차단 (override 4경로 · data 3 · 로그 원자료 6)

File: hanwha_robot_arm/HCR_5/hcr_robot_description/urdf/hcr_robot.ros2_control.xacro (robot description, xacro)
@@ -2,4 +2,45 @@
 <robot xmlns:xacro="http://www.ros.org/wiki/xacro">
   <!--
+    ══ 하드웨어 추상화 경계 ═══════════════════════════════════════════════════
+    sim 과 실기가 **같은 URDF 를 쓰고 플러그인만 갈아끼운다.** 셋 다 기본값이 있어
+    인자 없이 부르던 기존 사용처(display.launch.py · MoveIt2 demo)는 그대로 동작한다.
+      plugin    실기는 hcr5_bridge/HcrSystemInterface.
+                인자명을 동료 ysh 의 hcr5_description 과 맞춰 이식을 한 줄로 뒀다
+      rw_rate   이 하드웨어 컴포넌트만의 read()/write() 주기(Hz).
+                controller_manager 의 update_rate 와 분리된다 (ros2_control 4.45.2).
+                기본 100 = update_rate 와 같은 값이라 mock 거동이 종전과 같다.
+                ⚠️ 파서가 양의 정수를 요구한다 — 0 을 기본값으로 두면 뜨지 않는다
+      is_async  실기 명령 RPC 왕복이 115~137ms 라 동기 발행은 100Hz 루프를 막는다.
+                워커 스레드로 분리할 때 true
+    앞의 셋은 `<ros2_control>` **속성**이고, 아래 둘은 `<hardware>` 안의 **`<param>`** 이다.
+    ros2_control 이 둘을 다른 자리에서 읽으므로 실리는 곳이 다르다.
+      allow_motion  실기를 **실제로 움직일지**의 안전 잠금. 플러그인 기본값이 false 이고
+                    이 param 만이 켜는 유일한 통로다 (hcr_system_interface.cpp:108-118).
+                    false 면 write() 가 무동작 — 실기 '읽기 전용' 모드가 이 상태다.
+                    ⚠️ true 는 로봇이 움직인다. 서보 ON·e-stop 대기·입회를 갖추고서만 쓴다
+      servo_off_on_deactivate
+                    비활성화(= 종료)될 때 서보를 끌지. **기본 true.**
+                    allow_motion 과 무관하게 적용된다 — 읽기 전용으로 띄웠어도 서보는
+                    launch 나 사람이 켜 뒀을 수 있기 때문이다. mock 플러그인은 이 param 을
+                    안 읽으므로 mock 거동은 종전과 같다.
+                    ⚠️ false 로 두면 종료 후 서보가 켜진 채 남는다 — 축온이 올라
+                    58~61°C 에서 6축이 트립한다(2026-08-05, 컨트롤러 재부팅으로만 복구).
+                    자세가 위험해 브레이크를 걸고 싶지 않을 때만 false
+    실기 읽기는 `rw_rate:=30 is_async:=true` 로 연다 — 상태 버스 실측이 29.1Hz 다.
+    실기 쓰기는 거기에 `allow_motion:=true` 를 더한다.
+    근거: src/drivers/hcr5_comm/guideline/중간결과물.md §2·§5
+    ════════════════════════════════════════════════════════════════════════ -->
+  <xacro:macro name="hcr_robot_ros2_control"
+               params="name:=hcr_robot_system
+                       plugin:=mock_components/GenericSystem
+                       rw_rate:=100
+                       is_async:=false
+                       allow_motion:=false
+                       servo_off_on_deactivate:=true">
+    <ros2_control name="${name}" type="system" rw_rate="${rw_rate}" is_async="${is_async}">
+      <hardware>
+        <plugin>${plugin}</plugin>
+        <param name="allow_motion">${allow_motion}</param>
+        <param name="servo_off_on_deactivate">${servo_off_on_deactivate}</param>
       </hardware>
       <!-- initial_value = URDF 홈 [90, 0, 90, 0, 90, 0]°.

File: hanwha_robot_arm/HCR_5/hcr_robot_description/urdf/hcr_robot.xacro (robot description, xacro)
@@ -0,0 +1,271 @@
+<?xml version="1.0" ?>
+<robot name="hcr_robot" xmlns:xacro="http://www.ros.org/wiki/xacro">
+<!-- ── 인자 (하드웨어 추상화 경계) ────────────────────────────────────────────
+  선언을 **이 파일에** 두는 이유 — 이 URDF 를 읽는 진입점이 둘이다.
+    · hcr_robot_description/launch/display.launch.py  → 이 파일을 직접 읽는다
+    · hcr_moveit_config/config/hcr_robot.urdf.xacro   → 이 파일을 include 한다
+  기본값을 여기 두어야 두 경로가 다 산다. moveit 쪽에서 넘기는 mappings 가 이 기본값을 덮는다.
+    xacro hcr_robot.xacro                                          # mock (기본)
+    xacro hcr_robot.xacro hardware_plugin:=hcr5_bridge/HcrSystemInterface \
+                          rw_rate:=30 is_async:=true               # 실기 읽기
+    xacro hcr_robot.xacro hardware_plugin:=hcr5_bridge/HcrSystemInterface \
+                          rw_rate:=30 is_async:=true \
+                          allow_motion:=true                       # 실기 쓰기 ⚠️ 움직인다
+    xacro hcr_robot.xacro ros2_control:=false                      # 블록 생성 안 함
+  값의 의미·근거는 hcr_robot.ros2_control.xacro 머리말 -->
+<!-- ros2_control 블록을 아예 만들지 않는 갈래. 감싸는 쪽이 자체 블록을 정의할 때 쓴다
+     (시뮬레이션은 hardware 에 <param> 을 넣어야 해서 이 경로를 탄다 —
+      src/simulation/.../sim_bringup/urdf/hcr_robot_pen.xacro).
+     이 갈래가 없으면 mock 블록이 **항상** 들어가 다른 하드웨어와 같은 조인트를 두고 충돌한다. -->
+<xacro:arg name="ros2_control"    default="true"/>
+<xacro:arg name="hardware_plugin" default="mock_components/GenericSystem"/>
+<xacro:arg name="rw_rate"         default="100"/>
+<xacro:arg name="is_async"        default="false"/>
+<!-- 기본값 false 는 플러그인 기본값과 같다 — 인자를 잊어도 로봇은 안 움직인다 -->
+<xacro:arg name="allow_motion"    default="false"/>
+<xacro:arg name="servo_off_on_deactivate" default="true"/>
+<xacro:include filename="$(find hcr_robot_description)/urdf/materials.xacro" />
+<xacro:include filename="$(find hcr_robot_description)/urdf/hcr_robot.trans" />
+<xacro:include filename="$(find hcr_robot_description)/urdf/hcr_robot.gazebo" />
+<xacro:include filename="$(find hcr_robot_description)/urdf/hcr_robot.ros2_control.xacro" />
+<xacro:if value="$(arg ros2_control)">
+  <xacro:hcr_robot_ros2_control plugin="$(arg hardware_plugin)"
+                                rw_rate="$(arg rw_rate)"
+                                is_async="$(arg is_async)"
+                                allow_motion="$(arg allow_motion)"
+                                servo_off_on_deactivate="$(arg servo_off_on_deactivate)"/>
+</xacro:if>
+<link name="base_link">
+  <inertial>
+    <origin xyz="0.044693591972953806 -9.689819846991377e-05 0.013982771179495564" rpy="0 0 0"/>
+    <mass value="4.071462983655495"/>
+    <inertia ixx="0.004614" iyy="0.063084" izz="0.067151" ixy="-2e-05" iyz="0.0" ixz="-0.000189"/>
+  </inertial>
+  <visual>
+    <origin xyz="0 0 0" rpy="0 0 0"/>
+    <geometry>
+      <mesh filename="package://hcr_robot_description/meshes/base_link.stl" scale="0.001 0.001 0.001"/>
+    </geometry>
+    <material name="silver"/>
+  </visual>
+  <collision>
+    <origin xyz="0 0 0" rpy="0 0 0"/>
+    <geometry>
+      <mesh filename="package://hcr_robot_description/meshes/base_link.stl" scale="0.001 0.001 0.001"/>
+    </geometry>
+  </collision>
+</link>
+<link name="link1_1">
+  <inertial>
+    <origin xyz="-0.009232924655966162 5.611908895686318e-08 0.08981078121700108" rpy="0 0 0"/>
+    <mass value="17.125748524580114"/>
+    <inertia ixx="0.054601" iyy="0.061186" izz="0.036738" ixy="0.0" iyz="-0.0" ixz="0.004569"/>
+  </inertial>
+  <visual>
+    <origin xyz="-0.0 0.0 -0.03" rpy="0 0 0"/>
+    <geometry>
+      <mesh filename="package://hcr_robot_description/meshes/link1_1.stl" scale="0.001 0.001 0.001"/>
+    </geometry>
+    <material name="silver"/>
+  </visual>
+  <collision>
+    <origin xyz="-0.0 0.0 -0.03" rpy="0 0 0"/>
+    <geometry>
+      <mesh filename="package://hcr_robot_description/meshes/link1_1.stl" scale="0.001 0.001 0.001"/>
+    </geometry>
+  </collision>
+</link>
+<link name="link2_1">
+  <inertial>
+    <origin xyz="-0.08134423156498356 0.0004999972193747809 0.21200027982915884" rpy="0 0 0"/>
+    <mass value="32.073698785630135"/>
+    <inertia ixx="1.334728" iyy="1.368804" izz="0.0845" ixy="-5e-06" iyz="-0.003172" ixz="-0.002068"/>
+  </inertial>
+  <visual>
+    <origin xyz="0.0785 0.0 -0.148778" rpy="0 0 0"/>
+    <geometry>
+      <mesh filename="package://hcr_robot_description/meshes/link2_1.stl" scale="0.001 0.001 0.001"/>
+    </geometry>
+    <material name="silver"/>
+  </visual>
+  <collision>
+    <origin xyz="0.0785 0.0 -0.148778" rpy="0 0 0"/>
+    <geometry>
+      <mesh filename="package://hcr_robot_description/meshes/link2_1.stl" scale="0.001 0.001 0.001"/>
+    </geometry>
+  </collision>
+</link>
+<link name="link3_1">
+  <inertial>
+    <origin xyz="0.03733088153046067 -8.45436915776097e-06 0.32700293666580915" rpy="0 0 0"/>
+    <mass value="6.636542484506931"/>
+    <inertia ixx="0.008668" iyy="0.014027" izz="0.010649" ixy="-0.0" iyz="0.0" ixz="0.001661"/>
+  </inertial>
+  <visual>
+    <origin xyz="0.077848 -0.001 -0.572778" rpy="0 0 0"/>
+    <geometry>
+      <mesh filename="package://hcr_robot_description/meshes/link3_1.stl" scale="0.001 0.001 0.001"/>
+    </geometry>
+    <material name="silver"/>
+  </visual>
+  <collision>
+    <origin xyz="0.077848 -0.001 -0.572778" rpy="0 0 0"/>
+    <geometry>
+      <mesh filename="package://hcr_robot_description/meshes/link3_1.stl" scale="0.001 0.001 0.001"/>
+    </geometry>
+  </collision>
+</link>
+<link name="link4_1">
+  <inertial>
+    <origin xyz="-0.053462210233883714 -3.2261679182082545e-07 0.022076827880824546" rpy="0 0 0"/>
+    <mass value="6.518501202798632"/>
+    <inertia ixx="0.011005" iyy="0.012783" izz="0.007491" ixy="-0.0" iyz="0.0" ixz="0.001222"/>
+  </inertial>
+  <visual>
+    <origin xyz="0.107864 -0.000992 -0.911345" rpy="0 0 0"/>
+    <geometry>
+      <mesh filename="package://hcr_robot_description/meshes/link4_1.stl" scale="0.001 0.001 0.001"/>
+    </geometry>
+    <material name="silver"/>
+  </visual>
+  <collision>
+    <origin xyz="0.107864 -0.000992 -0.911345" rpy="0 0 0"/>
+    <geometry>
+      <mesh filename="package://hcr_robot_description/meshes/link4_1.stl" scale="0.001 0.001 0.001"/>
+    </geometry>
+  </collision>
+</link>
+<link name="link5_1">
+  <inertial>
+    <origin xyz="-0.022082116809040042 -5.860596366637823e-07 0.0534553107989999" rpy="0 0 0"/>
+    <mass value="6.518501237017786"/>
+    <inertia ixx="0.007541" iyy="0.012794" izz="0.010966" ixy="0.0" iyz="-0.0" ixz="0.001224"/>
+  </inertial>
+  <visual>
+    <origin xyz="0.169864 -0.000992 -1.000941" rpy="0 0 0"/>
+    <geometry>
+      <mesh filename="package://hcr_robot_description/meshes/link5_1.stl" scale="0.001 0.001 0.001"/>
+    </geometry>
+    <material name="silver"/>
+  </visual>
+  <collision>
+    <origin xyz="0.169864 -0.000992 -1.000941" rpy="0 0 0"/>
+    <geometry>
+      <mesh filename="package://hcr_robot_description/meshes/link5_1.stl" scale="0.001 0.001 0.001"/>
+    </geometry>
+  </collision>
+</link>
+<link name="link6_1">
+  <inertial>
+    <origin xyz="-0.019264152679962065 -4.5474100852818493e-07 -0.0005907014657897669" rpy="0 0 0"/>
+    <mass value="1.6914762668461325"/>
+    <inertia ixx="0.001473" iyy="0.00094" izz="0.000976" ixy="0.0" iyz="0.0" ixz="-8e-06"/>
+  </inertial>
+  <visual>
+    <origin xyz="0.25946 -0.000992 -1.062941" rpy="0 0 0"/>
+    <geometry>
+      <mesh filename="package://hcr_robot_description/meshes/link6_1.stl" scale="0.001 0.001 0.001"/>
+    </geometry>
+    <material name="silver"/>
+  </visual>
+  <collision>
+    <origin xyz="0.25946 -0.000992 -1.062941" rpy="0 0 0"/>
+    <geometry>
+      <mesh filename="package://hcr_robot_description/meshes/link6_1.stl" scale="0.001 0.001 0.001"/>
+    </geometry>
+  </collision>
+</link>
+<!-- ═══ 2026-08-05 실측 교정 ═══════════════════════════════════════════════════
+  실기(Rodi 1.003.005)의 FK RPC robot/convertPose 로 6축을 20°씩 전 회전 스윕(108샘플,
+  원적합 RMS 0.000mm)해 기구학을 추출하고 이 URDF 와 대조했다. 결과:
+  · origin 이 실기와 달랐다 (아래 ★ 표시 8곳). 특히 joint_6.x 의 42.9mm 오차가 지배적으로,
+    그것만 고쳐도 RMS 43.4mm → 1.6mm 로 떨어진다. 나머지는 1mm 이하의 미세 보정이다.
+    전부 적용 후 전 자세 위치오차 **RMS 43.4mm → 0.0060mm** (최대 0.0130mm, 109샘플 검증).
+  · limit 은 CAD 더미값(velocity=100 rad/s = 5729°/s)이었다. 매뉴얼 공식값으로 교체.
+  · 실기와 URDF 는 **영점 규약이 다르다**. 브릿지는 반드시 아래 변환을 적용할 것:
+        q_URDF[i] = s[i]*q_실기[i] + δ[i]      (도)
+        s = (+1, +1, −1, +1, +1, +1)          ← J3 만 부호 반전
+        δ = ( 90,  90,   0,  90,   0,   0)
+    실기 zero = 팔이 수평으로 뻗은 자세, URDF zero = 팔이 수직으로 선 자세.
+    실기 홈 [0,−90,−90,−90,90,0] = URDF [90,0,90,0,90,0] (SRDF hcr_home 과 일치시킴)
+  · mesh 는 CAD 기준 그대로다 — joint_6 을 42.9mm 옮겼으므로 시각화가 그만큼 어긋난다.
+    실기 제어에는 기구학 일치가 우선이라 이쪽을 택했다. mesh 교체는 별도 과제.
+  근거·재현: 업무목록 T16 · src/drivers/hcr5_mqtt/README.md
+════════════════════════════════════════════════════════════════════════════ -->
+<joint name="joint_1" type="revolute">
+  <origin xyz="0.0 0.0 0.03" rpy="0 0 0"/>
+  <parent link="base_link"/>
+  <child link="link1_1"/>
+  <axis xyz="0.0 -0.0 1.0"/>
+  <!-- 공식 ±360°, 180°/s (Appendix F·G). 종전 0~360°(음수 불가)는 IK 해가 있어도 계획 실패를 낳았다 -->
+  <!-- ★ 2026-08-15 교정 — 한계를 **실기 ±360° 에 정합**시켰다. 종전 URDF 대칭 ±360° 는
+       δ=90° 탓에 실기로는 [+270°, −450°] 라, 양(+)방향으로 **한 바퀴를 못 돌았다.**
+       실측: 실기 267.77° 에서 발행이 끊겼다 (URDF 360° = 실기 270° 벽).
+         upper  7.853981 ≈ URDF +450° = 실기 +360°
+         lower −4.712388 ≈ URDF −270° = 실기 −360°
+       ⚠️ 끝자리를 **안쪽으로 내렸다.** 정확한 450° 는 7.853981633974483 인데, 반올림한
+          `7.853982` 를 쓰면 실기 환산이 **360.000021°** 라 `withinLimits()`(실기 ±360°)에 걸린다 —
+          URDF 한계는 통과하는데 실기 검사가 막는 **게이트 충돌**이다. `-4.712389` 도 같다(−360.0000011°).
+          실측 2026-08-15: 목표 360° 가 이 경계에서 차단돼 **359.98° 에 멈췄다.**
+          URDF 한계는 실기 한계보다 **항상 안쪽**이어야 두 검사가 싸우지 않는다.
+       δ=90° 인 j1·j2·j4 가 같은 결함이었다. 근거: hcr5_bridge/운전절차.md §5 함정 ⑨ -->
+  <limit upper="7.853981" lower="-4.712388" effort="100" velocity="3.141593"/>
+</joint>
+<joint name="joint_2" type="revolute">
+  <!-- ★ 실측 교정: x −0.0785→−0.059138 (+19.36mm). joint_3.x 와 짝을 이룬다 (아래 참조) -->
+  <origin xyz="-0.059138 0.0 0.119001" rpy="0 0 0"/>
+  <parent link="link1_1"/>
+  <child link="link2_1"/>
+  <axis xyz="-1.0 0.0 0.0"/>
+  <!-- ★ 2026-08-15 교정 — δ=90° 정합. joint_1 주석 참조 -->
+  <limit upper="7.853981" lower="-4.712388" effort="100" velocity="3.141593"/>
+</joint>
+<joint name="joint_3" type="revolute">
+  <!-- ★ 실측 교정: z 0.424→0.425001 (상완 +1mm) · y 0.001→0 · x 0.000652→−0.019348
+       joint_2.x 와 joint_3.x 는 축이 평행해 겉보기엔 합만 의미 있을 것 같지만, 두 origin
+       사이에 J2 회전이 끼어 있어 실제로는 개별 식별된다. 합만 맞추면 RMS 가 0.28mm 로
+       남고, 최소제곱 해를 그대로 쓰면 0.0038mm 가 된다 -->
+  <origin xyz="-0.019348 0.0 0.425001" rpy="0 0 0"/>
+  <parent link="link2_1"/>
+  <child link="link3_1"/>
+  <axis xyz="1.0 0.0 0.0"/>
+  <!-- J3 만 별도 제한 ±165° 가 실제로 존재한다 -->
+  <limit upper="2.879793" lower="-2.879793" effort="100" velocity="3.141593"/>
+</joint>
+<joint name="joint_4" type="revolute">
+  <!-- ★ 실측 교정: z 0.338567→0.338499 (−0.07mm) -->
+  <origin xyz="-0.030016 -8e-06 0.338499" rpy="0 0 0"/>
+  <parent link="link3_1"/>
+  <child link="link4_1"/>
+  <axis xyz="-1.0 0.0 -0.0"/>
+  <!-- ★ 2026-08-15 교정 — δ=90° 정합. joint_1 주석 참조 -->
+  <limit upper="7.853981" lower="-4.712388" effort="100" velocity="3.141593"/>
+</joint>
+<joint name="joint_5" type="revolute">
+  <!-- ★ 실측 교정: z 0.089596→0.089504 (−0.09mm) -->
+  <origin xyz="-0.062 0.0 0.089504" rpy="0 0 0"/>
+  <parent link="link4_1"/>
+  <child link="link5_1"/>
+  <axis xyz="-0.0 -0.0 1.0"/>
+  <!-- 실기 wrist2 가 −267° 로 관측된다 — 종전 ±120° 로는 현재 자세조차 표현 못 했다 -->
+  <limit upper="6.283185" lower="-6.283185" effort="100" velocity="3.141593"/>
+</joint>
+<joint name="joint_6" type="revolute">
+  <!-- ★ 실측 교정: x −0.089596→−0.132498 (−42.90mm). J5 축에서 flange 까지 거리가
+       실기 132.5mm 인데 URDF 는 89.6mm 였다. 이 한 건이 전체 오차의 대부분이었다 -->
+  <origin xyz="-0.132498 0.0 0.062" rpy="0 0 0"/>
+  <parent link="link5_1"/>
+  <child link="link6_1"/>
+  <axis xyz="-1.0 -0.0 0.0"/>
+  <limit upper="6.283185" lower="-6.283185" effort="100" velocity="3.141593"/>
+</joint>
+<!-- ── 공구: 펜홀더 nyang_pen ─────────────────────────────────────────────────
+  플랜지(link6_1) 아래로 tool0 → 홀더 → 펜 → pen_tip 을 잇는다. pose goal 은
+  pen_tip 을 겨눈다 — 이 include 가 없으면 IK 가 **플랜지 기준**으로 풀린다.
+  본체와 분리된 패키지인 이유 · 명목 치수 · 강성 가정 · 축 방향 근거는 전부
+  src/drivers/nyang_pen/urdf/nyang_pen.xacro 머리말에 있다. 여기 옮겨 적지 않는다.
+  치수를 바꿀 때도 그 파일의 매크로 기본값만 고친다 (P1 판정 — 인자 관통 안 함).
+  ⚠️ 이 패키지는 compose.yml 이 src/drivers/ 를 마운트해야 컨테이너에서 보인다 -->
+<xacro:include filename="$(find nyang_pen)/urdf/nyang_pen.xacro"/>
+<xacro:nyang_pen parent="link6_1"/>
+</robot>
